Commit message: cambios11062020

File: irb120_robotiq85/irb120_robotiq85_gazebo/urdf/irb120_robotiq85_macro_final.xacro (robot description, xacro)
@@ -7,7 +7,4 @@
 	<!-- Robotiq 85 -->
 	<xacro:include filename="$(find robotiq_85_description)/urdf/robotiq_85_gripper.urdf.xacro" />
-	<!--xacro:robotiq_85_gripper prefix="" parent="tool0">
-		<origin xyz="0 0 0" rpy="0 0 0" />
-	</xacro:robotiq_85_gripper-->
 	<xacro:robotiq_85_gripper prefix="" parent="tool0">
 		<origin xyz="0 0 0" rpy="0 0 0" />
